File: hardware/D-Class_Amp/Input_Stage.sch (KiCad schematic (older format))
At the start: 0 parts

Commit message: Created the input filter schematic
Parts:
- added C? (x8): 100n, symbol Device:C
- added R? (x2): 5.6k, symbol Device:R
- added R? (x4): 8.2k, symbol Device:R
- added U? (x5): Opamp_Quad_Generic, symbol Device:Opamp_Quad_Generic
Connections:
- net labels added: +3.3V, -3V3, A_OUT, B_OUT, C_OUT, FILT_OUT, GND, GNDS, SIG_IN
- wire segments 0 -> 57
