File: hardware/D-Class_Amp/Input_Stage.sch (KiCad schematic (older format))
At the start: 21 parts, among them U201 LM324

Commit message: fixed the inout filter gain stage
Parts:
- C202: symbol D-Class_Amp-rescue:CP_Small-Device -> Device:CP_Small
- RV201: symbol D-Class_Amp-rescue:R_POT-Device -> Device:R_POT
Connections:
- net +2V5: now also RV201.3; no longer R204.2
- net C_OUT: now also R204.2, TP202.1; no longer R204.1, RV201.3
- net at RV201.2, U201.9 (-): now also R204.1; no longer TP202.1
- no-connect marks 1 -> 0
Other:
- moved on the sheet: C201, C202, C203, C204, C205, C206, C207, C208, JP201, R201, R202, R203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
