File: hardware/D-Class_Amp/Power_Stage.sch (KiCad schematic (older format))
At the start: 0 parts

Commit message: added parts
Parts:
- added C? (x2): C_Small, symbol Device:C_Small
- added Q? (x4): Q_NMOS_GDSD, symbol Device:Q_NMOS_GDSD
- added R? (x6): R, symbol Device:R
- added U? (x2): IR21834, symbol Driver_FET:IR21834
Connections:
- new net S-PWM: U?.1 (HIN), U?.2 (~LIN)
Changed lines of the file:
@@
 $Descr A4 11693 8268
 encoding utf-8
-Sheet 1 4
+Sheet 1 1
 Title ""
 Date ""
@@
 Comment4 ""
 $EndDescr
+$Comp
+L Driver_FET:IR21834 U?
+U 1 1 6104C522
+P 4200 2600
+F 0 "U?" H 4200 3281 50  0000 C CNN
+F 1 "IR21834" H 4200 3190 50  0000 C CNN
+F 2 "" H 4200 2600 50  0001 C CIN
+F 3 "https://www.infineon.com/dgdl/ir2183.pdf?fileId=5546d462533600a4015355c9490e16d1" H 4200 2600 50  0001 C CNN
+	1    4200 2600
+	1    0    0    -1
+$EndComp
+$Comp
+L Driver_FET:IR21834 U?
+U 1 1 6104CE13
+P 4200 4600
+F 0 "U?" H 4200 5281 50  0000 C CNN
+F 1 "IR21834" H 4200 5190 50  0000 C CNN
+F 2 "" H 4200 4600 50  0001 C CIN
+F 3 "https://www.infineon.com/dgdl/ir2183.pdf?fileId=5546d462533600a4015355c9490e16d1" H 4200 4600 50  0001 C CNN
+	1    4200 4600
+	1    0    0    -1
+$EndComp
+$Comp
+L Device:Q_NMOS_GDSD Q?
+U 1 1 6104F024
+P 5400 2050
+F 0 "Q?" H 5688 2096 50  0000 L CNN
+F 1 "Q_NMOS_GDSD" H 5688 2005 50  0000 L CNN
+F 2 "" H 5600 2150 50  0001 C CNN
+F 3 "~" H 5400 2050 50  0001 C CNN
+	1    5400 2050
+	1    0    0    -1
+$EndComp
+$Comp
+L Device:Q_NMOS_GDSD Q?
+U 1 1 6104F394
+P 5450 3050
+F 0 "Q?" H 5738 3096 50  0000 L CNN
+F 1 "Q_NMOS_GDSD" H 5738 3005 50  0000 L CNN
+F 2 "" H 5650 3150 50  0001 C CNN
+F 3 "~" H 5450 3050 50  0001 C CNN
+	1    5450 3050
+	1    0    0    -1
+$EndComp
+$Comp
+L Device:Q_NMOS_GDSD Q?
+U 1 1 6104FAFA
+P 5500 4950
+F 0 "Q?" H 5788 4996 50  0000 L CNN
+F 1 "Q_NMOS_GDSD" H 5788 4905 50  0000 L CNN
+F 2 "" H 5700 5050 50  0001 C CNN
+F 3 "~" H 5500 4950 50  0001 C CNN
+	1    5500 4950
+	1    0    0    -1
+$EndComp
+$Comp
+L Device:Q_NMOS_GDSD Q?
+U 1 1 6104FB04
+P 5550 4200
+F 0 "Q?" H 5838 4246 50  0000 L CNN
+F 1 "Q_NMOS_GDSD" H 5838 4155 50  0000 L CNN
+F 2 "" H 5750 4300 50  0001 C CNN
+F 3 "~" H 5550 4200 50  0001 C CNN
+	1    5550 4200
+	1    0    0    -1
+$EndComp
+$Comp
+L Device:R R?
+U 1 1 61051377
+P 5000 2400
+F 0 "R?" H 5070 2446 50  0000 L CNN
+F 1 "R" H 5070 2355 50  0000 L CNN
+F 2 "" V 4930 2400 50  0001 C CNN
+F 3 "~" H 5000 2400 50  0001 C CNN
+	1    5000 2400
+	1    0    0    -1
+$EndComp
+$Comp
+L Device:R R?
+U 1 1 61051734
+P 4950 4950
+F 0 "R?" H 5020 4996 50  0000 L CNN
+F 1 "R" H 5020 4905 50  0000 L CNN
+F 2 "" V 4880 4950 50  0001 C CNN
+F 3 "~" H 4950 4950 50  0001 C CNN
+	1    4950 4950
+	1    0    0    -1
+$EndComp
+$Comp
+L Device:R R?
+U 1 1 61052B3F
+P 5000 4200
+F 0 "R?" H 5070 4246 50  0000 L CNN
+F 1 "R" H 5070 4155 50  0000 L CNN
+F 2 "" V 4930 4200 50  0001 C CNN
+F 3 "~" H 5000 4200 50  0001 C CNN
+	1    5000 4200
+	1    0    0    -1
+$EndComp
+$Comp
+L Device:R R?
+U 1 1 610540BF
+P 5050 3050
+F 0 "R?" H 5120 3096 50  0000 L CNN
+F 1 "R" H 5120 3005 50  0000 L CNN
+F 2 "" V 4980 3050 50  0001 C CNN
+F 3 "~" H 5050 3050 50  0001 C CNN
+	1    5050 3050
+	1    0    0    -1
+$EndComp
+$Comp
+L Device:R R?
+U 1 1 61055141
+P 3700 2800
+F 0 "R?" V 3600 2800 50  0000 C CNN
+F 1 "R" V 3500 2800 50  0000 C CNN
+F 2 "" V 3630 2800 50  0001 C CNN
+F 3 "~" H 3700 2800 50  0001 C CNN
+	1    3700 2800
+	0    -1   -1   0
+$EndComp
+$Comp
+L power:VDD #PWR?
+U 1 1 6105D8A1
+P 2300 1600
+F 0 "#PWR?" H 2300 1450 50  0001 C CNN
+F 1 "VDD" H 2315 1773 50  0000 C CNN
+F 2 "" H 2300 1600 50  0001 C CNN
+F 3 "" H 2300 1600 50  0001 C CNN
+	1    2300 1600
+	1    0    0    -1
+$EndComp
+$Comp
+L power:GND #PWR?
+U 1 1 6105F7B4
+P 3400 1750
+F 0 "#PWR?" H 3400 1500 50  0001 C CNN
+F 1 "GND" H 3405 1577 50  0000 C CNN
+F 2 "" H 3400 1750 50  0001 C CNN
+F 3 "" H 3400 1750 50  0001 C CNN
+	1    3400 1750
+	1    0    0    -1
+$EndComp
+$Comp
+L power:VSS #PWR?
+U 1 1 6105E48C
+P 2300 1800
+F 0 "#PWR?" H 2300 1650 50  0001 C CNN
+F 1 "VSS" H 2315 1973 50  0000 C CNN
+F 2 "" H 2300 1800 50  0001 C CNN
+F 3 "" H 2300 1800 50  0001 C CNN
+	1    2300 1800
+	-1   0    0    1
+$EndComp
+$Comp
+L Device:R R?
+U 1 1 61067213
+P 3400 4450
+F 0 "R?" H 3470 4496 50  0000 L CNN
+F 1 "R" H 3470 4405 50  0000 L CNN
+F 2 "" V 3330 4450 50  0001 C CNN
+F 3 "~" H 3400 4450 50  0001 C CNN
+	1    3400 4450
+	1    0    0    -1
+$EndComp
+Text HLabel 3800 2600 0    50   Input ~ 0
+S-PWM
+Text HLabel 3650 4850 0    50   Input ~ 0
+~S-PWM
+Text HLabel 6600 2550 0    50   Output ~ 0
+P_OUT
+Text HLabel 6650 4550 0    50   Output ~ 0
+~P_OUT
+$Comp
+L Device:C_Small C?
+U 1 1 610A4CCB
+P 4750 1850
+F 0 "C?" H 4842 1896 50  0000 L CNN
+F 1 "C_Small" H 4842 1805 50  0000 L CNN
+F 2 "" H 4750 1850 50  0001 C CNN
+F 3 "~" H 4750 1850 50  0001 C CNN
+	1    4750 1850
+	1    0    0    -1
+$EndComp
+$Comp
+L Device:C_Small C?
+U 1 1 610A52A3
+P 4700 4050
+F 0 "C?" H 4792 4096 50  0000 L CNN
+F 1 "C_Small" H 4792 4005 50  0000 L CNN
+F 2 "" H 4700 4050 50  0001 C CNN
+F 3 "~" H 4700 4050 50  0001 C CNN
+	1    4700 4050
+	1    0    0    -1
+$EndComp
+$Comp
+L power:+12V #PWR?
+U 1 1 610ABD74
+P 3600 1550
+F 0 "#PWR?" H 3600 1400 50  0001 C CNN
+F 1 "+12V" H 3615 1723 50  0000 C CNN
+F 2 "" H 3600 1550 50  0001 C CNN
+F 3 "" H 3600 1550 50  0001 C CNN
+	1    3600 1550
+	1    0    0    -1
+$EndComp
+Wire Wire Line
+	3800 2600 3850 2600
+Wire Wire Line
+	3850 2600 3850 2700
+Wire Wire Line
+	3850 2700 3900 2700
+Connection ~ 3850 2600
+Wire Wire Line
+	3850 2600 3900 2600
 $EndSCHEMATC
