File: hardware/D-Class_Amp/Power_Stage.sch (KiCad schematic (older format))
At the start: 22 parts, among them Q501 PHP23NQ11T, Q502 PHP23NQ11T, Q503 PHP23NQ11T, Q504 PHP23NQ11T, U501 IR21834, U502 IR21834

Commit message: Designed the triangle generator PCB layout, and the power switching stage layout
Parts:
- Q501, Q502, Q503, Q504: footprint Package_TO_SOT_THT:TO-251-3-1EP_Horizontal_TabDown -> PHP23NQ11T:PHP23NQ11T
Changed lines of the file:
@@
 F 0 "Q501" H 6038 1346 50  0000 L CNN
 F 1 "PHP23NQ11T" H 6038 1255 50  0000 L CNN
-F 2 "Package_TO_SOT_THT:TO-251-3-1EP_Horizontal_TabDown" H 5950 1400 50  0001 C CNN
+F 2 "PHP23NQ11T:PHP23NQ11T" H 5950 1400 50  0001 C CNN
 F 3 "https://assets.nexperia.com/documents/data-sheet/PHP23NQ11T.pdf" H 5750 1300 50  0001 C CNN
 F 4 "1.90" H 5750 1300 50  0001 C CNN "DigiKey Price"
@@
 	0    1    1    0
 $EndComp
+Wire Wire Line
+	4950 825  4950 1300
+Connection ~ 4950 1300
+Wire Wire Line
+	4950 1300 5200 1300
+Wire Wire Line
+	4550 1800 5175 1800
+Connection ~ 5175 1800
+Wire Wire Line
+	5175 1800 5200 1800
+Wire Wire Line
+	5175 1025 5175 1800
+Wire Wire Line
+	9050 1025 9050 1300
+Wire Wire Line
+	9275 825  9275 1800
+Connection ~ 9050 1300
+Wire Wire Line
+	9050 1300 9000 1300
+Connection ~ 9275 1800
+Wire Wire Line
+	9275 1800 9000 1800
+$Comp
+L Device:Q_NMOS_GDSD Q502
+U 1 1 61187A5E
+P 5750 1800
+F 0 "Q502" H 6038 1846 50  0000 L CNN
+F 1 "PHP23NQ11T" H 6038 1755 50  0000 L CNN
+F 2 "PHP23NQ11T:PHP23NQ11T" H 5950 1900 50  0001 C CNN
+F 3 "https://assets.nexperia.com/documents/data-sheet/PHP23NQ11T.pdf" H 5750 1800 50  0001 C CNN
+F 4 "1.90" H 5750 1800 50  0001 C CNN "DigiKey Price"
+F 5 "PHP23NQ11T,127" H 5750 1800 50  0001 C CNN "Part Number"
+	1    5750 1800
+	1    0    0    -1
+$EndComp
+Wire Wire Line
+	8350 1550 8350 1500
+$Comp
+L Device:Q_NMOS_GDSD Q503
+U 1 1 6118B010
+P 8450 1300
+F 0 "Q503" H 8738 1346 50  0000 L CNN
+F 1 "PHP23NQ11T" H 8738 1255 50  0000 L CNN
+F 2 "PHP23NQ11T:PHP23NQ11T" H 8650 1400 50  0001 C CNN
+F 3 "https://assets.nexperia.com/documents/data-sheet/PHP23NQ11T.pdf" H 8450 1300 50  0001 C CNN
+F 4 "1.90" H 8450 1300 50  0001 C CNN "DigiKey Price"
+F 5 "PHP23NQ11T,127" H 8450 1300 50  0001 C CNN "Part Number"
+	1    8450 1300
+	-1   0    0    -1
+$EndComp
+$Comp
+L Device:Q_NMOS_GDSD Q504
+U 1 1 6118BB1D
+P 8450 1800
+F 0 "Q504" H 8738 1846 50  0000 L CNN
+F 1 "PHP23NQ11T" H 8738 1755 50  0000 L CNN
+F 2 "PHP23NQ11T:PHP23NQ11T" H 8650 1900 50  0001 C CNN
+F 3 "https://assets.nexperia.com/documents/data-sheet/PHP23NQ11T.pdf" H 8450 1800 50  0001 C CNN
+F 4 "1.90" H 8450 1800 50  0001 C CNN "DigiKey Price"
+F 5 "PHP23NQ11T,127" H 8450 1800 50  0001 C CNN "Part Number"
+	1    8450 1800
+	-1   0    0    -1
+$EndComp
+$Comp
+L Device:C_Small C501
+U 1 1 61199493
+P 3550 1275
+F 0 "C501" H 3275 1350 50  0000 L CNN
+F 1 "10u 16V" H 3150 1275 50  0000 L CNN
+F 2 "Capacitor_SMD:C_0805_2012Metric_Pad1.18x1.45mm_HandSolder" H 3550 1275 50  0001 C CNN
+F 3 "~" H 3550 1275 50  0001 C CNN
+F 4 "0.34" H 3550 1275 50  0001 C CNN "DigiKey Price"
+F 5 "CL21A106KOQNNWE" H 3550 1275 50  0001 C CNN "Part Number"
+	1    3550 1275
+	1    0    0    -1
+$EndComp
+$Comp
+L Device:C_Small C504
+U 1 1 6119B46C
+P 10650 1275
+F 0 "C504" H 10375 1350 50  0000 L CNN
+F 1 "10u 16V" H 10250 1275 50  0000 L CNN
+F 2 "Capacitor_SMD:C_0805_2012Metric_Pad1.18x1.45mm_HandSolder" H 10650 1275 50  0001 C CNN
+F 3 "~" H 10650 1275 50  0001 C CNN
+F 4 "0.34" H 10650 1275 50  0001 C CNN "DigiKey Price"
+F 5 "CL21A106KOQNNWE" H 10650 1275 50  0001 C CNN "Part Number"
+	1    10650 1275
+	-1   0    0    -1
+$EndComp
+Wire Wire Line
+	10650 1700 10650 1375
+Connection ~ 10650 1700
+Wire Wire Line
+	10650 1175 10650 950
+Wire Wire Line
+	10650 950  9950 950
+Wire Wire Line
+	4250 950  3550 950
+Wire Wire Line
+	3550 950  3550 1175
+Wire Wire Line
+	3550 1375 3550 1700
+Connection ~ 3550 1700
+$Comp
+L Connector:TestPoint TP?
+U 1 1 61153163
+P 9275 825
+AR Path="/61153163" Ref="TP?"  Part="1"
+AR Path="/610497A4/61153163" Ref="TP504"  Part="1"
+F 0 "TP504" H 8975 1000 50  0000 L CNN
+F 1 "~LO" H 9225 1050 50  0000 L CNN
+F 2 "TestPoint:TestPoint_THTPad_D2.0mm_Drill1.0mm" H 9475 825 50  0001 C CNN
+F 3 "~" H 9475 825 50  0001 C CNN
+	1    9275 825
+	1    0    0    -1
+$EndComp
+$Comp
+L Connector:TestPoint TP?
+U 1 1 61152F83
+P 9050 1025
+AR Path="/61152F83" Ref="TP?"  Part="1"
+AR Path="/610497A4/61152F83" Ref="TP503"  Part="1"
+F 0 "TP503" H 8775 1150 50  0000 L CNN
+F 1 "~HO" H 9000 1250 50  0000 L CNN
+F 2 "TestPoint:TestPoint_THTPad_D2.0mm_Drill1.0mm" H 9250 1025 50  0001 C CNN
+F 3 "~" H 9250 1025 50  0001 C CNN
+	1    9050 1025
+	1    0    0    -1
+$EndComp
+$Comp
+L Connector:TestPoint TP?
+U 1 1 6114A61F
+P 5175 1025
+AR Path="/6114A61F" Ref="TP?"  Part="1"
+AR Path="/610497A4/6114A61F" Ref="TP502"  Part="1"
+F 0 "TP502" H 5233 1149 50  0000 L CNN
+F 1 "LO" H 5125 1250 50  0000 L CNN
+F 2 "TestPoint:TestPoint_THTPad_D2.0mm_Drill1.0mm" H 5375 1025 50  0001 C CNN
+F 3 "~" H 5375 1025 50  0001 C CNN
+	1    5175 1025
+	1    0    0    -1
+$EndComp
 $Comp
 L Connector:TestPoint TP?
@@
 	1    0    0    -1
 $EndComp
-$Comp
-L Connector:TestPoint TP?
-U 1 1 6114A61F
-P 5175 1025
-AR Path="/6114A61F" Ref="TP?"  Part="1"
-AR Path="/610497A4/6114A61F" Ref="TP502"  Part="1"
-F 0 "TP502" H 5233 1149 50  0000 L CNN
-F 1 "LO" H 5125 1250 50  0000 L CNN
-F 2 "TestPoint:TestPoint_THTPad_D2.0mm_Drill1.0mm" H 5375 1025 50  0001 C CNN
-F 3 "~" H 5375 1025 50  0001 C CNN
-	1    5175 1025
-	1    0    0    -1
-$EndComp
-Wire Wire Line
-	4950 825  4950 1300
-Connection ~ 4950 1300
-Wire Wire Line
-	4950 1300 5200 1300
-Wire Wire Line
-	4550 1800 5175 1800
-Connection ~ 5175 1800
-Wire Wire Line
-	5175 1800 5200 1800
-Wire Wire Line
-	5175 1025 5175 1800
-$Comp
-L Connector:TestPoint TP?
-U 1 1 61152F83
-P 9050 1025
-AR Path="/61152F83" Ref="TP?"  Part="1"
-AR Path="/610497A4/61152F83" Ref="TP503"  Part="1"
-F 0 "TP503" H 8775 1150 50  0000 L CNN
-F 1 "~HO" H 9000 1250 50  0000 L CNN
-F 2 "TestPoint:TestPoint_THTPad_D2.0mm_Drill1.0mm" H 9250 1025 50  0001 C CNN
-F 3 "~" H 9250 1025 50  0001 C CNN
-	1    9050 1025
-	1    0    0    -1
-$EndComp
-$Comp
-L Connector:TestPoint TP?
-U 1 1 61153163
-P 9275 825
-AR Path="/61153163" Ref="TP?"  Part="1"
-AR Path="/610497A4/61153163" Ref="TP504"  Part="1"
-F 0 "TP504" H 8975 1000 50  0000 L CNN
-F 1 "~LO" H 9225 1050 50  0000 L CNN
-F 2 "TestPoint:TestPoint_THTPad_D2.0mm_Drill1.0mm" H 9475 825 50  0001 C CNN
-F 3 "~" H 9475 825 50  0001 C CNN
-	1    9275 825
-	1    0    0    -1
-$EndComp
-Wire Wire Line
-	9050 1025 9050 1300
-Wire Wire Line
-	9275 825  9275 1800
-Connection ~ 9050 1300
-Wire Wire Line
-	9050 1300 9000 1300
-Connection ~ 9275 1800
-Wire Wire Line
-	9275 1800 9000 1800
-$Comp
-L Device:Q_NMOS_GDSD Q502
-U 1 1 61187A5E
-P 5750 1800
-F 0 "Q502" H 6038 1846 50  0000 L CNN
-F 1 "PHP23NQ11T" H 6038 1755 50  0000 L CNN
-F 2 "Package_TO_SOT_THT:TO-251-3-1EP_Horizontal_TabDown" H 5950 1900 50  0001 C CNN
-F 3 "https://assets.nexperia.com/documents/data-sheet/PHP23NQ11T.pdf" H 5750 1800 50  0001 C CNN
-F 4 "1.90" H 5750 1800 50  0001 C CNN "DigiKey Price"
-F 5 "PHP23NQ11T,127" H 5750 1800 50  0001 C CNN "Part Number"
-	1    5750 1800
-	1    0    0    -1
-$EndComp
-Wire Wire Line
-	8350 1550 8350 1500
-$Comp
-L Device:Q_NMOS_GDSD Q503
-U 1 1 6118B010
-P 8450 1300
-F 0 "Q503" H 8738 1346 50  0000 L CNN
-F 1 "PHP23NQ11T" H 8738 1255 50  0000 L CNN
-F 2 "Package_TO_SOT_THT:TO-251-3-1EP_Horizontal_TabDown" H 8650 1400 50  0001 C CNN
-F 3 "https://assets.nexperia.com/documents/data-sheet/PHP23NQ11T.pdf" H 8450 1300 50  0001 C CNN
-F 4 "1.90" H 8450 1300 50  0001 C CNN "DigiKey Price"
-F 5 "PHP23NQ11T,127" H 8450 1300 50  0001 C CNN "Part Number"
-	1    8450 1300
-	-1   0    0    -1
-$EndComp
-$Comp
-L Device:Q_NMOS_GDSD Q504
-U 1 1 6118BB1D
-P 8450 1800
-F 0 "Q504" H 8738 1846 50  0000 L CNN
-F 1 "PHP23NQ11T" H 8738 1755 50  0000 L CNN
-F 2 "Package_TO_SOT_THT:TO-251-3-1EP_Horizontal_TabDown" H 8650 1900 50  0001 C CNN
-F 3 "https://assets.nexperia.com/documents/data-sheet/PHP23NQ11T.pdf" H 8450 1800 50  0001 C CNN
-F 4 "1.90" H 8450 1800 50  0001 C CNN "DigiKey Price"
-F 5 "PHP23NQ11T,127" H 8450 1800 50  0001 C CNN "Part Number"
-	1    8450 1800
-	-1   0    0    -1
-$EndComp
-$Comp
-L Device:C_Small C501
-U 1 1 61199493
-P 3550 1275
-F 0 "C501" H 3275 1350 50  0000 L CNN
-F 1 "10u 16V" H 3150 1275 50  0000 L CNN
-F 2 "Capacitor_SMD:C_0805_2012Metric_Pad1.18x1.45mm_HandSolder" H 3550 1275 50  0001 C CNN
-F 3 "~" H 3550 1275 50  0001 C CNN
-F 4 "0.34" H 3550 1275 50  0001 C CNN "DigiKey Price"
-F 5 "CL21A106KOQNNWE" H 3550 1275 50  0001 C CNN "Part Number"
-	1    3550 1275
-	1    0    0    -1
-$EndComp
-$Comp
-L Device:C_Small C504
-U 1 1 6119B46C
-P 10650 1275
-F 0 "C504" H 10375 1350 50  0000 L CNN
-F 1 "10u 16V" H 10250 1275 50  0000 L CNN
-F 2 "Capacitor_SMD:C_0805_2012Metric_Pad1.18x1.45mm_HandSolder" H 10650 1275 50  0001 C CNN
-F 3 "~" H 10650 1275 50  0001 C CNN
-F 4 "0.34" H 10650 1275 50  0001 C CNN "DigiKey Price"
-F 5 "CL21A106KOQNNWE" H 10650 1275 50  0001 C CNN "Part Number"
-	1    10650 1275
-	-1   0    0    -1
-$EndComp
-Wire Wire Line
-	10650 1700 10650 1375
-Connection ~ 10650 1700
-Wire Wire Line
-	10650 1175 10650 950
-Wire Wire Line
-	10650 950  9950 950
-Wire Wire Line
-	4250 950  3550 950
-Wire Wire Line
-	3550 950  3550 1175
-Wire Wire Line
-	3550 1375 3550 1700
-Connection ~ 3550 1700
 $EndSCHEMATC

Commit message: placed and routed all components, fixed the MOSFET footprints, and added all 3D models.
Parts:
- TP501, TP502, TP503, TP504: footprint TestPoint:TestPoint_THTPad_D2.0mm_Drill1.0mm -> TestPoint:TestPoint_THTPad_D1.0mm_Drill0.5mm
Changed lines of the file:
@@
 F 0 "TP504" H 8975 1000 50  0000 L CNN
 F 1 "~LO" H 9225 1050 50  0000 L CNN
-F 2 "TestPoint:TestPoint_THTPad_D2.0mm_Drill1.0mm" H 9475 825 50  0001 C CNN
+F 2 "TestPoint:TestPoint_THTPad_D1.0mm_Drill0.5mm" H 9475 825 50  0001 C CNN
 F 3 "~" H 9475 825 50  0001 C CNN
 	1    9275 825
@@
 F 0 "TP503" H 8775 1150 50  0000 L CNN
 F 1 "~HO" H 9000 1250 50  0000 L CNN
-F 2 "TestPoint:TestPoint_THTPad_D2.0mm_Drill1.0mm" H 9250 1025 50  0001 C CNN
+F 2 "TestPoint:TestPoint_THTPad_D1.0mm_Drill0.5mm" H 9250 1025 50  0001 C CNN
 F 3 "~" H 9250 1025 50  0001 C CNN
 	1    9050 1025
@@
 F 0 "TP502" H 5233 1149 50  0000 L CNN
 F 1 "LO" H 5125 1250 50  0000 L CNN
-F 2 "TestPoint:TestPoint_THTPad_D2.0mm_Drill1.0mm" H 5375 1025 50  0001 C CNN
+F 2 "TestPoint:TestPoint_THTPad_D1.0mm_Drill0.5mm" H 5375 1025 50  0001 C CNN
 F 3 "~" H 5375 1025 50  0001 C CNN
 	1    5175 1025
@@
 F 0 "TP501" H 5008 949 50  0000 L CNN
 F 1 "HO" H 4900 1050 50  0000 L CNN
-F 2 "TestPoint:TestPoint_THTPad_D2.0mm_Drill1.0mm" H 5150 825 50  0001 C CNN
+F 2 "TestPoint:TestPoint_THTPad_D1.0mm_Drill0.5mm" H 5150 825 50  0001 C CNN
 F 3 "~" H 5150 825 50  0001 C CNN
 	1    4950 825
