File: hardware/D-Class_Amp/D-Class_Amp.kicad_pcb (KiCad board)
At the start: 2 copper layers, 84 parts, among them J102 AudioJack2, Q501 PHP23NQ11T, Q502 PHP23NQ11T, Q503 PHP23NQ11T, Q504 PHP23NQ11T, U101 NCP1117-12_TO252, U102 MCP1799T-5002H_TT, U201 LM324, U301 TL972, U302 LMV393, U501 IR21834, U502 IR21834

Commit message: REGION CITY
Parts:
- moved TP109 55.0 mm to (116.5, 57.0)
- moved TP110 55.0 mm to (116.5, 52.9)
- moved TP504 50.2 mm to (88.9, 51.3)
- moved TP503 48.0 mm to (94.7, 53.1)
- moved TP103 46.2 mm to (19.7, 70.9)
- moved TP201 46.2 mm to (24.6, 71.1)
- moved C104 45.3 mm to (78.1, 104.9), turned to 90 degrees
- moved TP104 35.5 mm to (53.3, 54.6)
- moved TP301 34.7 mm to (40.4, 55.0)
- moved TP302 34.7 mm to (40.3, 49.7)
- moved TP102 34.2 mm to (62.6, 69.0)
- moved TP105 33.6 mm to (69.8, 50.8)
- moved TP101 30.4 mm to (107.2, 69.1)
- moved TP108 29.9 mm to (75.4, 53.6)
- moved TP106 29.5 mm to (59.9, 51.6)
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Routing:
- net +12V: track 37.0 -> 60.8 mm
- net VDD: track 0.00 -> 8.89 mm
- added copper zone on F.Cu, net /Output_Filter/SPEAKER_OUT
- added copper zone on F.Cu, net /Output_Filter/~SPEAKER_OUT
- added copper zone on B.Cu, net /Power_Stage/P_OUT
- added copper zone on F.Cu, net /Power_Stage/P_OUT
- added copper zone on B.Cu, net /Power_Stage/~P_OUT
- added copper zone on F.Cu, net /Power_Stage/~P_OUT
- added copper zone on B.Cu, net GND
