File: hardware/D-Class_Amp/D-Class_Amp.sch (KiCad schematic (older format))
At the start: 31 parts, among them J101 P_IN, J102 AudioJack2, U101 NCP1117-12_TO252, U102 MCP1799T-5002H_TT

Commit message: created a bill of materials
Parts:
- C104: Part Number (none) -> UVR1H102MHD1TO
Changed lines of the file:
@@
 F 3 "~" H 3450 2550 50  0001 C CNN
 F 4 "1" H 3450 2550 50  0001 C CNN "DigiKey Price"
+F 5 "UVR1H102MHD1TO" H 3450 2550 50  0001 C CNN "Part Number"
 	1    3450 2550
 	0    -1   -1   0

Commit message: update design
Parts:
- added C?: 100u, Capacitor_SMD:CP_Elec_4x5.4, symbol Device:CP_Small
Connections:
- net +2V5: now also C?.1
- net GNDS: now also C?.2
Other:
- moved on the sheet: C103, C105, R101, R102, U102

Commit message: res cap to ref
Parts:
- gave numbers to parts that had none: 1
Changed lines of the file:
@@
 P 4150 1450
 AR Path="/610497A4/616826E8" Ref="C?"  Part="1"
-AR Path="/616826E8" Ref="C?"  Part="1"
-F 0 "C?" H 3975 1450 50  0000 L CNN
+AR Path="/616826E8" Ref="C106"  Part="1"
+F 0 "C106" H 3900 1450 50  0000 L CNN
 F 1 "100u" H 3900 1375 50  0000 L CNN
 F 2 "Capacitor_SMD:CP_Elec_4x5.4" H 4150 1450 50  0001 C CNN

Commit message: teardrop ref cap, regen BOM
Parts:
- C106: value 100u -> 100n 16V
Changed lines of the file:
@@
 AR Path="/610497A4/616826E8" Ref="C?"  Part="1"
 AR Path="/616826E8" Ref="C106"  Part="1"
-F 0 "C106" H 3900 1450 50  0000 L CNN
-F 1 "100u" H 3900 1375 50  0000 L CNN
+F 0 "C106" H 3875 1450 50  0000 L CNN
+F 1 "100n 16V" H 3875 1375 50  0000 L CNN
 F 2 "Capacitor_SMD:CP_Elec_4x5.4" H 4150 1450 50  0001 C CNN
 F 3 "~" H 4150 1450 50  0001 C CNN
